Commit message: 添加URDF

File: so101_9_28.urdf (robot description, URDF)
Before this commit: robot so101_new_calib, 8 links, 7 joints
Links:
- link gripper_link: geometry collision box size=0.0022 0.008 0.01; collision box size=0.003 0.012 0.01
- link moving_jaw_so101_v1_link: geometry collision box size=0.002 0.01 0.008; collision box size=0.002 0.01 0.012
